File: hardware/BusinessCard/BusinessCard.kicad_pcb (KiCad board)
At the start: 2 copper layers, 88.9 x 50.8 mm, 5 parts, among them U2 NT3H2211W0FHKH

Commit message: fix: invalid pcb comment
Other:
- board text removed: "0.2000 mm / 0.2000 mm"
- board text removed: "0.3000 mm"
- board text removed: "1.6000 mm"
- board text removed: "100.0000 mm x 100.0000 mm"
- board text removed: "BOARD CHARACTERISTICS"
- board text removed: "Board Thickness:"
- board text removed: "Board overall dimensions:"
- board text removed: "Castellated pads:"
- board text removed: "Copper Finish:"
- board text removed: "Copper Layer Count:"
- board text removed: "ENIG"
- board text removed: "Edge card connectors:"
- board text removed: "Impedance Control:"
- board text removed: "Min hole diameter:"
- board text removed: "Min track/spacing:"
- board text removed: "No"
- board text removed: "Plated Board Edge:"
